Commit message: URDF file updated with new sensor configuration.

File: src/robot_model/urdf/robot.urdf.xacro (robot description, xacro)
@@ -105,34 +105,66 @@
         <limit lower="0.0" upper="0.03" effort="50" velocity="2"/>
     </joint>
-    <!-- Left Gripper -->
-    <link name="left_gripper_wheel">
+      <!-- ================= GRIPPER MACRO ================= -->
+    <xacro:macro name="gripper" params="name x y yaw">
+      <link name="${name}">
         <visual>
-            <geometry>
+          <origin rpy="1.5708 0 0"/>
+          <geometry>
             <cylinder radius="0.015" length="0.03"/>
-            </geometry>
-            <material name="black"/>
+          </geometry>
+          <material name="black">
+            <color rgba="0 0 0 1"/>
+          </material>
         </visual>
-    </link>
-    <joint name="left_gripper_joint" type="continuous">
+        <collision>
+          <origin rpy="1.5708 0 0"/>
+          <geometry>
+            <cylinder radius="0.015" length="0.03"/>
+          </geometry>
+        </collision>
+        <inertial>
+          <mass value="0.05"/>
+          <inertia
+            ixx="0.00002" ixy="0" ixz="0"
+            iyy="0.00002" iyz="0"
+            izz="0.00002"/>
+        </inertial>
+      </link>
+      <joint name="${name}_joint" type="continuous">
         <parent link="base_link"/>
-        <child link="left_gripper_wheel"/>
-        <origin xyz="0.2 0.04 0.04"/>
+        <child link="${name}"/>
+        <origin xyz="${x} ${y} 0.04" rpy="0 0 ${yaw}"/>
         <axis xyz="0 1 0"/>
-    </joint>
-    <!-- Right Gripper -->
-    <link name="right_gripper_wheel">
-        <visual>
-            <geometry>
-            <cylinder radius="0.015" length="0.03"/>
-            </geometry>
-            <material name="black"/>
-        </visual>
-    </link>
-    <joint name="right_gripper_joint" type="continuous">
-        <parent link="base_link"/>
-        <child link="right_gripper_wheel"/>
-        <origin xyz="0.2 -0.04 0.04"/>
-        <axis xyz="0 1 0"/>
-    </joint>
+      </joint>
+    </xacro:macro>
+      <!-- ================= GRIPPERS ================= -->
+    <xacro:gripper name="left_gripper_wheel"  x="0.2"  y="0.05" yaw="-0.3"/>
+    <xacro:gripper name="right_gripper_wheel" x="0.2"  y="-0.05" yaw="0.3"/>
+  <!-- ================= LIDAR ================= -->
+  <link name="lidar_link">
+    <visual>
+      <geometry>
+        <cylinder radius="0.03" length="0.03"/>
+      </geometry>
+      <material name="black"/>
+    </visual>
+    <collision>
+      <geometry>
+        <cylinder radius="0.03" length="0.03"/>
+      </geometry>
+    </collision>
+    <inertial>
+      <mass value="0.1"/>
+      <inertia
+        ixx="0.0001" ixy="0" ixz="0"
+        iyy="0.0001" iyz="0"
+        izz="0.0001"/>
+    </inertial>
+  </link>
+  <joint name="lidar_joint" type="fixed">
+    <parent link="base_link"/>
+    <child link="lidar_link"/>
+    <origin xyz="0 0 0.115" rpy="0 0 0"/>
+  </joint>
     <!-- Gazebo Condition -->
   <gazebo reference="base_link">
@@ -163,3 +195,53 @@
     <selfCollide>false</selfCollide>
     </gazebo>
+<!--Lidar Gazebo-->
+      <gazebo reference="lidar_link">
+    <sensor type="ray" name="lidar">
+      <pose>0 0 0 0 0 0</pose>
+      <update_rate>20</update_rate>
+      <ray>
+        <scan>
+          <horizontal>
+            <samples>720</samples>
+            <min_angle>-3.14159</min_angle>
+            <max_angle>3.14159</max_angle>
+          </horizontal>
+        </scan>
+        <range>
+          <min>0.05</min>
+          <max>6.0</max>
+        </range>
+      </ray>
+      <plugin name="gazebo_ros_laser" filename="libgazebo_ros_laser.so">
+        <topicName>/scan</topicName>
+        <frameName>lidar_link</frameName>
+      </plugin>
+    </sensor>
+  </gazebo>
+  <!-- Wheels Friction Gazebo -->
+  <gazebo reference="front_left_wheel">
+    <mu1>1.2</mu1>
+    <mu2>1.2</mu2>
+  </gazebo>
+  <gazebo reference="front_right_wheel">
+    <mu1>1.2</mu1>
+    <mu2>1.2</mu2>
+  </gazebo>
+  <gazebo reference="back_left_wheel">
+    <mu1>1.2</mu1>
+    <mu2>1.2</mu2>
+  </gazebo>
+  <gazebo reference="back_right_wheel">
+    <mu1>1.2</mu1>
+    <mu2>1.2</mu2>
+  </gazebo>
+  <!-- Gripper Friction Gazebo -->
+  <gazebo reference="left_gripper_wheel">
+    <mu1>1.2</mu1>
+    <mu2>1.2</mu2>
+  </gazebo>
+  <gazebo reference="right_gripper_wheel">
+    <mu1>1.2</mu1>
+    <mu2>1.2</mu2>
+  </gazebo>
 </robot>

Commit message: URDF Added Lidar, Solenoid, Camera and gripper

File: src/robot_model/urdf/robot.urdf.xacro (robot description, xacro)
@@ -67,5 +67,6 @@
       <child link="${name}"/>
       <origin xyz="${x} ${y} 0.0"/>
-      <axis xyz="0 1 0"/>
+      <axis xyz="0 0 1"/>
+      <dynamics damping="0.1" friction="0.0"/>
     </joint>
   </xacro:macro>
@@ -221,19 +222,43 @@
   <!-- Wheels Friction Gazebo -->
   <gazebo reference="front_left_wheel">
-    <mu1>1.2</mu1>
-    <mu2>1.2</mu2>
-  </gazebo>
+  <surface>
+    <friction>
+      <ode>
+        <mu>1.2</mu>
+        <mu2>1.2</mu2>
+      </ode>
+    </friction>
+  </surface>
+</gazebo>
   <gazebo reference="front_right_wheel">
-    <mu1>1.2</mu1>
-    <mu2>1.2</mu2>
-  </gazebo>
+  <surface>
+    <friction>
+      <ode>
+        <mu>1.2</mu>
+        <mu2>1.2</mu2>
+      </ode>
+    </friction>
+  </surface>
+</gazebo>
   <gazebo reference="back_left_wheel">
-    <mu1>1.2</mu1>
-    <mu2>1.2</mu2>
-  </gazebo>
+  <surface>
+    <friction>
+      <ode>
+        <mu>1.2</mu>
+        <mu2>1.2</mu2>
+      </ode>
+    </friction>
+  </surface>
+</gazebo>
   <gazebo reference="back_right_wheel">
-    <mu1>1.2</mu1>
-    <mu2>1.2</mu2>
-  </gazebo>
+  <surface>
+    <friction>
+      <ode>
+        <mu>1.2</mu>
+        <mu2>1.2</mu2>
+      </ode>
+    </friction>
+  </surface>
+</gazebo>
   <!-- Gripper Friction Gazebo -->
   <gazebo reference="left_gripper_wheel">
@@ -245,3 +270,29 @@
     <mu2>1.2</mu2>
   </gazebo>
+  <gazebo>
+  <plugin name="diff_drive" filename="libgazebo_ros_diff_drive.so">
+    <leftJoint>front_left_wheel_joint back_left_wheel_joint</leftJoint>
+    <rightJoint>front_right_wheel_joint back_right_wheel_joint</rightJoint>
+    <wheelSeparation>0.30</wheelSeparation>
+    <wheelDiameter>0.06</wheelDiameter>
+    <robotBaseFrame>base_link</robotBaseFrame>
+    <odomFrame>odom</odomFrame>
+    <topicName>cmd_vel</topicName>
+    <odometryTopic>odom</odometryTopic>
+  </plugin>
+</gazebo>
+<gazebo reference="camera_link">
+  <sensor type="camera" name="camera">
+    <camera>
+      <horizontal_fov>1.047</horizontal_fov>
+      <image>
+        <width>640</width>
+        <height>480</height>
+      </image>
+    </camera>
+    <plugin name="gazebo_ros_camera" filename="libgazebo_ros_camera.so">
+      <frameName>camera_link</frameName>
+    </plugin>
+  </sensor>
+</gazebo>
 </robot>

Commit message: Update URDF and launch files for improved robot simulation setup

File: src/robot_model/urdf/robot.urdf.xacro (robot description, xacro)
@@ -67,5 +67,5 @@
       <child link="${name}"/>
       <origin xyz="${x} ${y} 0.0"/>
-      <axis xyz="0 0 1"/>
+      <axis xyz="0 1 0"/>
       <dynamics damping="0.1" friction="0.0"/>
     </joint>
@@ -198,26 +198,23 @@
 <!--Lidar Gazebo-->
       <gazebo reference="lidar_link">
-    <sensor type="ray" name="lidar">
-      <pose>0 0 0 0 0 0</pose>
-      <update_rate>20</update_rate>
-      <ray>
-        <scan>
-          <horizontal>
-            <samples>720</samples>
-            <min_angle>-3.14159</min_angle>
-            <max_angle>3.14159</max_angle>
-          </horizontal>
-        </scan>
-        <range>
-          <min>0.05</min>
-          <max>6.0</max>
-        </range>
-      </ray>
-      <plugin name="gazebo_ros_laser" filename="libgazebo_ros_laser.so">
-        <topicName>/scan</topicName>
-        <frameName>lidar_link</frameName>
-      </plugin>
-    </sensor>
-  </gazebo>
+  <sensor name="lidar" type="gpu_lidar">
+    <pose>0 0 0 0 0 0</pose>
+    <update_rate>20</update_rate>
+    <ray>
+      <scan>
+        <horizontal>
+          <samples>720</samples>
+          <min_angle>-3.14159</min_angle>
+          <max_angle>3.14159</max_angle>
+        </horizontal>
+      </scan>
+      <range>
+        <min>0.05</min>
+        <max>6.0</max>
+      </range>
+    </ray>
+    <topic>/scan</topic>
+  </sensor>
+</gazebo>
   <!-- Wheels Friction Gazebo -->
   <gazebo reference="front_left_wheel">
@@ -271,17 +268,23 @@
   </gazebo>
   <gazebo>
-  <plugin name="diff_drive" filename="libgazebo_ros_diff_drive.so">
-    <leftJoint>front_left_wheel_joint back_left_wheel_joint</leftJoint>
-    <rightJoint>front_right_wheel_joint back_right_wheel_joint</rightJoint>
-    <wheelSeparation>0.30</wheelSeparation>
-    <wheelDiameter>0.06</wheelDiameter>
-    <robotBaseFrame>base_link</robotBaseFrame>
-    <odomFrame>odom</odomFrame>
-    <topicName>cmd_vel</topicName>
-    <odometryTopic>odom</odometryTopic>
+  <plugin
+    filename="gz-sim-diff-drive-system"
+    name="gz::sim::systems::DiffDrive">
+    <left_joint>front_left_wheel_joint</left_joint>
+    <left_joint>back_left_wheel_joint</left_joint>
+    <right_joint>front_right_wheel_joint</right_joint>
+    <right_joint>back_right_wheel_joint</right_joint>
+    <wheel_separation>0.30</wheel_separation>
+    <wheel_radius>0.03</wheel_radius>
+    <odom_publish_frequency>50</odom_publish_frequency>
+    <topic>cmd_vel</topic>
+    <odom_topic>odom</odom_topic>
+    <frame_id>odom</frame_id>
+    <child_frame_id>base_link</child_frame_id>
   </plugin>
 </gazebo>
 <gazebo reference="camera_link">
-  <sensor type="camera" name="camera">
+  <sensor name="camera" type="camera">
+    <pose>0 0 0 0 0 0</pose>
     <camera>
       <horizontal_fov>1.047</horizontal_fov>
@@ -289,9 +292,12 @@
         <width>640</width>
         <height>480</height>
+        <format>R8G8B8</format>
       </image>
+      <clip>
+        <near>0.1</near>
+        <far>100</far>
+      </clip>
     </camera>
-    <plugin name="gazebo_ros_camera" filename="libgazebo_ros_camera.so">
-      <frameName>camera_link</frameName>
-    </plugin>
+    <topic>/camera/image</topic>
   </sensor>
 </gazebo>

Commit message: Refactor launch file and URDF for improved robot simulation; add lidar model

File: src/robot_model/urdf/robot.urdf.xacro (robot description, xacro)
@@ -78,15 +78,15 @@
     <!-- Camera -->
     <link name="camera_link">
-        <visual>
-            <geometry>
-            <box size="0.02 0.02 0.02"/>
-            </geometry>
-            <material name="blue"/>
-        </visual>
+      <visual>
+        <geometry>
+          <box size="0.02 0.02 0.02"/>
+        </geometry>
+        <material name="blue"/>
+      </visual>
     </link>
     <joint name="camera_joint" type="fixed">
-        <parent link="base_link"/>
-        <child link="camera_link"/>
-        <origin xyz="0.18 0 0.11" rpy="0 0 0"/>
+      <parent link="base_link"/>
+      <child link="camera_link"/>
+      <origin xyz="0.18 0 0.11" rpy="0 0 0"/>
     </joint>
     <!-- Kicker (solenoid valve) -->
@@ -98,4 +98,12 @@
             <material name="gray"/>
         </visual>
+      <inertial>
+        <origin xyz="0 0 0"/>
+        <mass value="0.1"/>
+        <inertia
+          ixx="0.0001" ixy="0.0" ixz="0.0"
+          iyy="0.0001" iyz="0.0"
+          izz="0.0001"/>
+      </inertial>
     </link>
     <joint name="kicker_joint" type="prismatic">
@@ -139,5 +147,5 @@
       </joint>
     </xacro:macro>
-      <!-- ================= GRIPPERS ================= -->
+  <!-- ================= GRIPPERS ================= -->
     <xacro:gripper name="left_gripper_wheel"  x="0.2"  y="0.05" yaw="-0.3"/>
     <xacro:gripper name="right_gripper_wheel" x="0.2"  y="-0.05" yaw="0.3"/>
@@ -166,5 +174,5 @@
     <parent link="base_link"/>
     <child link="lidar_link"/>
-    <origin xyz="0 0 0.115" rpy="0 0 0"/>
+    <origin xyz="0 0 0.116" rpy="0 0 0"/>
   </joint>
     <!-- Gazebo Condition -->
@@ -196,9 +204,15 @@
     <selfCollide>false</selfCollide>
     </gazebo>
+  <gazebo reference="lidar_link">
+    <selfCollide>false</selfCollide>
+    </gazebo>
+    <!-- LIDAR Sensor -->
     <gazebo reference="lidar_link">
-      <sensor name="lidar" type="gpu_lidar">
-        <pose>0 0 0 0 0 0</pose>
+      <sensor name="lidar" type="ray">
+        <always_on>true</always_on>
+        <visualize>true</visualize>
         <update_rate>20</update_rate>
-        <lidar>
+        <enable_collision>true</enable_collision>
+        <ray>
           <scan>
             <horizontal>
@@ -212,50 +226,26 @@
             <max>6.0</max>
           </range>
-        </lidar>
-        <!-- Gazebo transport topic -->
+        </ray>
         <topic>/scan</topic>
       </sensor>
     </gazebo>
-  <!-- Wheels Friction Gazebo -->
-  <gazebo reference="front_left_wheel">
-  <surface>
-    <friction>
-      <ode>
-        <mu>1.2</mu>
-        <mu2>1.2</mu2>
-      </ode>
-    </friction>
-  </surface>
-</gazebo>
-  <gazebo reference="front_right_wheel">
-  <surface>
-    <friction>
-      <ode>
-        <mu>1.2</mu>
-        <mu2>1.2</mu2>
-      </ode>
-    </friction>
-  </surface>
-</gazebo>
-  <gazebo reference="back_left_wheel">
-  <surface>
-    <friction>
-      <ode>
-        <mu>1.2</mu>
-        <mu2>1.2</mu2>
-      </ode>
-    </friction>
-  </surface>
-</gazebo>
-  <gazebo reference="back_right_wheel">
-  <surface>
-    <friction>
-      <ode>
-        <mu>1.2</mu>
-        <mu2>1.2</mu2>
-      </ode>
-    </friction>
-  </surface>
-</gazebo>
+  <!-- Wheel Friction Macro -->
+  <xacro:macro name="wheel_friction" params="wheel">
+  <gazebo reference="${wheel}">
+    <surface>
+      <friction>
+        <ode>
+          <mu>1.2</mu>
+          <mu2>1.2</mu2>
+        </ode>
+      </friction>
+    </surface>
+  </gazebo>
+</xacro:macro>
+<!-- Apply friction to all wheels -->
+<xacro:wheel_friction wheel="front_left_wheel"/>
+<xacro:wheel_friction wheel="front_right_wheel"/>
+<xacro:wheel_friction wheel="back_left_wheel"/>
+<xacro:wheel_friction wheel="back_right_wheel"/>
   <!-- Gripper Friction Gazebo -->
   <gazebo reference="left_gripper_wheel">
@@ -267,38 +257,48 @@
     <mu2>1.2</mu2>
   </gazebo>
+  <!-- Diff Drive Plugin -->
   <gazebo>
-  <plugin
-    filename="gz-sim-diff-drive-system"
-    name="gz::sim::systems::DiffDrive">
-    <left_joint>front_left_wheel_joint</left_joint>
-    <left_joint>back_left_wheel_joint</left_joint>
-    <right_joint>front_right_wheel_joint</right_joint>
-    <right_joint>back_right_wheel_joint</right_joint>
-    <wheel_separation>0.30</wheel_separation>
-    <wheel_radius>0.03</wheel_radius>
-    <odom_publish_frequency>50</odom_publish_frequency>
-    <topic>cmd_vel</topic>
-    <odom_topic>odom</odom_topic>
-    <frame_id>odom</frame_id>
-    <child_frame_id>base_link</child_frame_id>
+    <plugin
+      filename="gz-sim-diff-drive-system"
+      name="gz::sim::systems::DiffDrive">
+      <left_joint>front_left_wheel_joint</left_joint>
+      <left_joint>back_left_wheel_joint</left_joint>
+      <right_joint>front_right_wheel_joint</right_joint>
+      <right_joint>back_right_wheel_joint</right_joint>
+      <wheel_separation>0.30</wheel_separation>
+      <wheel_radius>0.03</wheel_radius>
+      <odom_publish_frequency>50</odom_publish_frequency>
+      <topic>cmd_vel</topic>
+      <odom_topic>odom</odom_topic>
+      <frame_id>odom</frame_id>
+      <child_frame_id>base_link</child_frame_id>
   </plugin>
 </gazebo>
+<!-- Sensors Plugin -->
+<gazebo>
+    <plugin
+      filename="gz-sim-sensors-system"
+      name="gz::sim::systems::Sensors"/>
+</gazebo>
+<!-- Gazebo Sensor for Camera -->
 <gazebo reference="camera_link">
-  <sensor name="camera" type="camera">
-    <pose>0 0 0 0 0 0</pose>
-    <camera>
-      <horizontal_fov>1.047</horizontal_fov>
-      <image>
-        <width>640</width>
-        <height>480</height>
-        <format>R8G8B8</format>
-      </image>
-      <clip>
-        <near>0.1</near>
-        <far>100</far>
-      </clip>
-    </camera>
-    <topic>/camera/image</topic>
-  </sensor>
-</gazebo>
+    <sensor name="camera" type="camera">
+      <always_on>true</always_on>
+      <visualize>true</visualize>
+      <update_rate>30</update_rate>
+      <camera>
+        <horizontal_fov>1.047</horizontal_fov>
+        <image>
+          <width>640</width>
+          <height>480</height>
+          <format>R8G8B8</format>
+        </image>
+        <clip>
+          <near>0.1</near>
+          <far>100</far>
+        </clip>
+      </camera>
+      <topic>/camera/image</topic>
+    </sensor>
+  </gazebo>
 </robot>

Commit message: Update Gazebo launch configuration and robot URDF model
- Adjusted the soccer bot's launch parameters to change the z-coordinate from 0.1 to 0.2 for better positioning.
- Added optional pose parameters for the soccer ball model, including x, y, z positions and roll, pitch, yaw orientations.
- Changed the robot's visual material from gray to black in the URDF model.
- Updated LIDAR sensor type from 'ray' to 'gpu_lidar' and modified its parameters, including reducing the horizontal samples from 720 to 360 and increasing the maximum range from 6.0 to 10.0 meters.
- Added a new graph file to visualize the robot's frame transformations and generated a PDF representation of the frames.

File: src/robot_model/urdf/robot.urdf.xacro (robot description, xacro)
@@ -96,5 +96,5 @@
             <box size="0.05 0.02 0.01"/>
             </geometry>
-            <material name="gray"/>
+            <material name="black"/>
         </visual>
       <inertial>
@@ -209,13 +209,14 @@
     <!-- LIDAR Sensor -->
     <gazebo reference="lidar_link">
-      <sensor name="lidar" type="ray">
+      <sensor name="lidar" type="gpu_lidar">
         <always_on>true</always_on>
+        <update_rate>10</update_rate>
         <visualize>true</visualize>
-        <update_rate>20</update_rate>
-        <enable_collision>true</enable_collision>
-        <ray>
+        <topic>scan</topic>
+        <lidar>
           <scan>
             <horizontal>
-              <samples>720</samples>
+              <samples>360</samples>
+              <resolution>1</resolution>
               <min_angle>-3.14159</min_angle>
               <max_angle>3.14159</max_angle>
@@ -224,8 +225,8 @@
           <range>
             <min>0.05</min>
-            <max>6.0</max>
+            <max>10.0</max>
+            <resolution>0.01</resolution>
           </range>
-        </ray>
-        <topic>/scan</topic>
+        </lidar>
       </sensor>
     </gazebo>

Commit message: Implement ball chasing functionality with dynamic HSV tuning. Add IMU and IR sensor to robot model URDF

File: src/robot_model/urdf/robot.urdf.xacro (robot description, xacro)
@@ -37,4 +37,42 @@
     </inertial>
   </link>
+  <!-- IMU LINK -->
+  <link name="imu_link">
+    <visual>
+      <geometry>
+        <box size="0.01 0.01 0.01"/>
+      </geometry>
+      <material name="red"/>
+    </visual>
+    <collision>
+      <geometry>
+        <box size="0.01 0.01 0.01"/>
+      </geometry>
+    </collision>
+    <inertial>
+      <mass value="0.01"/>
+      <inertia
+        ixx="1e-5" ixy="0" ixz="0"
+        iyy="1e-5" iyz="0"
+        izz="1e-5"/>
+    </inertial>
+  </link>
+  <joint name="imu_joint" type="fixed">
+    <parent link="base_link"/>
+    <child link="imu_link"/>
+    <origin xyz="0 0 0.137"/>
+  </joint>
+  <!-- IR SENSOR LINK -->
+  <link name="ir_link">
+    <inertial>
+      <mass value="0.005"/>
+      <inertia ixx="1e-6" iyy="1e-6" izz="1e-6"/>
+    </inertial>
+  </link>
+  <joint name="ir_joint" type="fixed">
+    <parent link="base_link"/>
+    <child link="ir_link"/>
+    <origin xyz="0.22 0 0.03"/>
+  </joint>
   <!-- ================= WHEEL MACRO ================= -->
   <xacro:macro name="wheel" params="name x y">
@@ -207,4 +245,7 @@
     <selfCollide>false</selfCollide>
     </gazebo>
+  <gazebo reference="imu_link">
+    <selfCollide>false</selfCollide>
+    </gazebo>
     <!-- LIDAR Sensor -->
     <gazebo reference="lidar_link">
@@ -281,4 +322,7 @@
       filename="gz-sim-sensors-system"
       name="gz::sim::systems::Sensors"/>
+    <plugin
+      filename="gz-sim-imu-system"
+      name="gz::sim::systems::Imu"/>
 </gazebo>
 <!-- Gazebo Sensor for Camera -->
@@ -303,3 +347,45 @@
     </sensor>
   </gazebo>
+  <!-- Gazebo Sensor for IMU -->
+  <gazebo reference="base_link">
+    <sensor name="imu_sensor" type="imu">
+      <always_on>true</always_on>
+      <update_rate>200</update_rate>
+      <visualize>false</visualize>
+      <topic>/imu/data</topic>
+      <imu>
+        <angular_velocity>
+          <x><noise type="gaussian"><mean>0</mean><stddev>0.00001</stddev></noise></x>
+          <y><noise type="gaussian"><mean>0</mean><stddev>0.00001</stddev></noise></y>
+          <z><noise type="gaussian"><mean>0</mean><stddev>0.00001</stddev></noise></z>
+        </angular_velocity>
+        <linear_acceleration>
+          <x><noise type="gaussian"><mean>0</mean><stddev>0.001</stddev></noise></x>
+          <y><noise type="gaussian"><mean>0</mean><stddev>0.001</stddev></noise></y>
+          <z><noise type="gaussian"><mean>0</mean><stddev>0.001</stddev></noise></z>
+        </linear_acceleration>
+      </imu>
+    </sensor>
+  </gazebo>
+  <!-- Gazebo Sensor for IR -->
+  <gazebo reference="ir_link">
+    <sensor name="ir_sensor" type="gpu_lidar">
+      <always_on>true</always_on>
+      <update_rate>50</update_rate>
+      <topic>/ir/beam</topic>
+      <lidar>
+        <scan>
+          <horizontal>
+            <samples>1</samples>
+            <min_angle>0</min_angle>
+            <max_angle>0</max_angle>
+          </horizontal>
+        </scan>
+        <range>
+          <min>0.01</min>
+          <max>0.15</max>
+        </range>
+      </lidar>
+    </sensor>
+  </gazebo>
 </robot>

Commit message: modify src/robot_model/urdf/robot.urdf.xacro

File: src/robot_model/urdf/robot.urdf.xacro (robot description, xacro)
@@ -69,9 +69,20 @@
       <inertia ixx="1e-6" iyy="1e-6" izz="1e-6"/>
     </inertial>
+    <visual>
+      <geometry>
+        <cylinder radius="0.005" length="0.02"/>
+      </geometry>
+      <material name="green"/>
+    </visual>
+    <collision>
+      <geometry>
+        <cylinder radius="0.005" length="0.02"/>
+      </geometry>
+    </collision>
   </link>
   <joint name="ir_joint" type="fixed">
     <parent link="base_link"/>
     <child link="ir_link"/>
-    <origin xyz="0.22 0 0.03"/>
+    <origin xyz="0.22 0 0.049"/>
   </joint>
   <!-- ================= WHEEL MACRO ================= -->
@@ -248,4 +259,7 @@
     <selfCollide>false</selfCollide>
     </gazebo>
+  <gazebo reference="ir_link">
+    <selfCollide>false</selfCollide>
+    </gazebo>
     <!-- LIDAR Sensor -->
     <gazebo reference="lidar_link">
@@ -384,5 +398,5 @@
         <range>
           <min>0.01</min>
-          <max>0.15</max>
+          <max>0.02</max>
         </range>
       </lidar>
